File: ScholDigi.kicad_pcb (KiCad board)
At the start: 2 copper layers, 66 x 49 mm, 67 parts, among them J1 Conn_01x04, J2 USB_C_Receptacle_USB2.0_14P, J3 Battery JST, J4 GPS Antenna coaxial, J5 USB_C_Receptacle_USB2.0_14P, Q1 FS8205A, SW1 Boot Button, SW2 Reset Button, U1 ESP32-C6-MINI-1, U2 MAX-M10S, U3 TP4056-42-ESOP8, U4 DW01A, U5 TPS63060, U6 CP2102

Commit message: small changes
Parts:
- J1: footprint Connector_Wire:SolderWire-0.1sqmm_1x04_P3.6mm_D0.4mm_OD1mm -> Connector_Wire:SolderWire-0.5sqmm_1x04_P4.6mm_D0.9mm_OD2.1mm
- moved J1 2.42 mm to (93.5, 60.0)
Routing:
- net IO2: track 6.74 -> 5.79 mm
- net VIN-: track 349.5 -> 350.2 mm
Changed lines of the file:
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@@
 		)
 	)
-	(footprint "Connector_Wire:SolderWire-0.1sqmm_1x04_P3.6mm_D0.4mm_OD1mm"
+	(footprint "Connector_Wire:SolderWire-0.5sqmm_1x04_P4.6mm_D0.9mm_OD2.1mm"
 		(layer "F.Cu")
-		(at 95.825 59.325)
-		(descr "Soldered wire connection, for 4 times 0.1 mm² wires, basic insulation, conductor diameter 0.4mm, outer diameter 1mm, size source Multi-Contact FLEXI-E 0.10 (https://www.staubli.com/content/dam/ecs/catalogs-brochures/TM/CAB-Main-11014119-en.pdf#page=9), bend radius 3 times outer diameter")
-		(tags "connector wire 0.1sqmm")
+		(at 93.5 60)
+		(descr "Soldered wire connection, for 4 times 0.5 mm² wires, basic insulation, conductor diameter 0.9mm, outer diameter 2.1mm, size source Multi-Contact FLEXI-E 0.50 (https://www.staubli.com/content/dam/ecs/catalogs-brochures/TM/CAB-Main-11014119-en.pdf#page=9), bend radius 3 times outer diameter")
+		(tags "connector wire 0.5sqmm")
 		(property "Reference" "J1"
-			(at -2.325 2.175 0)
+			(at 6.9 -2.28 0)
 			(layer "F.SilkS")
 			(effects
@@
 		)
 		(property "Value" "Conn_01x04"
-			(at -2.325 -3.325 90)
+			(at 6.9 2.28 0)
 			(layer "F.Fab")
 			(effects
@@
 		(duplicate_pad_numbers_are_jumpers no)
 		(fp_rect
-			(start -1.3 -1.3)
-			(end 1.3 1.3)
+			(start -1.8 -1.58)
+			(end 1.8 1.58)
 			(stroke
 				(width 0.05)
@@
 		)
 		(fp_rect
-			(start 2.3 -1.3)
-			(end 4.9 1.3)
+			(start 2.8 -1.58)
+			(end 6.4 1.58)
 			(stroke
 				(width 0.05)
@@
 		)
 		(fp_rect
-			(start 5.9 -1.3)
-			(end 8.5 1.3)
+			(start 7.4 -1.58)
+			(end 11 1.58)
 			(stroke
 				(width 0.05)
@@
 		)
 		(fp_rect
-			(start 9.5 -1.3)
-			(end 12.1 1.3)
+			(start 12 -1.58)
+			(end 15.6 1.58)
 			(stroke
 				(width 0.05)
@@
 		(fp_circle
 			(center 0 0)
-			(end 0.5 0)
+			(end 1.05 0)
 			(stroke
 				(width 0.1)
@@
 		)
 		(fp_circle
-			(center 3.6 0)
-			(end 4.1 0)
+			(center 4.6 0)
+			(end 5.65 0)
 			(stroke
 				(width 0.1)
@@
 		)
 		(fp_circle
-			(center 7.2 0)
-			(end 7.7 0)
+			(center 9.2 0)
+			(end 10.25 0)
 			(stroke
 				(width 0.1)
@@
 		)
 		(fp_circle
-			(center 10.8 0)
-			(end 11.3 0)
+			(center 13.8 0)
+			(end 14.85 0)
 			(stroke
 				(width 0.1)
@@
 		)
 		(fp_text user "${REFERENCE}"
-			(at 5.4 0 90)
+			(at 6.9 0 90)
 			(layer "F.Fab")
 			(effects
 				(font
-					(size 0.65 0.65)
-					(thickness 0.1)
+					(size 0.79 0.79)
+					(thickness 0.12)
 				)
 			)
@@
 		(pad "1" thru_hole roundrect
 			(at 0 0)
-			(size 1.6 1.6)
-			(drill 0.6)
+			(size 2.15 2.15)
+			(drill 1.15)
 			(layers "*.Cu" "*.Mask")
 			(remove_unused_layers no)
-			(roundrect_rratio 0.15625)
+			(roundrect_rratio 0.116279)
 			(net "VIN-")
 			(pinfunction "Pin_1_1")
@@
 		)
 		(pad "2" thru_hole circle
-			(at 3.6 0)
-			(size 1.6 1.6)
-			(drill 0.6)
+			(at 4.6 0)
+			(size 2.15 2.15)
+			(drill 1.15)
 			(layers "*.Cu" "*.Mask")
 			(remove_unused_layers no)
@@
 		)
 		(pad "3" thru_hole circle
-			(at 7.2 0)
-			(size 1.6 1.6)
-			(drill 0.6)
+			(at 9.2 0)
+			(size 2.15 2.15)
+			(drill 1.15)
 			(layers "*.Cu" "*.Mask")
 			(remove_unused_layers no)
@@
 		)
 		(pad "4" thru_hole circle
-			(at 10.8 0)
-			(size 1.6 1.6)
-			(drill 0.6)
+			(at 13.8 0)
+			(size 2.15 2.15)
+			(drill 1.15)
 			(layers "*.Cu" "*.Mask")
 			(remove_unused_layers no)
@@
 		)
 		(embedded_fonts no)
-		(model "${KICAD10_3DMODEL_DIR}/Connector_Wire.3dshapes/SolderWire-0.1sqmm_1x04_P3.6mm_D0.4mm_OD1mm.step"
+		(model "${KICAD10_3DMODEL_DIR}/Connector_Wire.3dshapes/SolderWire-0.5sqmm_1x04_P4.6mm_D0.9mm_OD2.1mm.step"
 			(offset
 				(xyz 0 0 0)
@@
 	)
 	(gr_text "IO3"
-		(at 102 62 0)
+		(at 101.5 63 0)
 		(layer "F.SilkS")
 		(effects
@@
 	)
 	(gr_text "IO2"
-		(at 105.5 62 0)
+		(at 106.5 63 0)
 		(layer "F.SilkS")
 		(effects
@@
 	)
 	(gr_text "GND"
-		(at 94.5 62 0)
+		(at 92 63 0)
 		(layer "F.SilkS")
 		(effects
@@
 	)
 	(gr_text "3v3"
-		(at 98.5 62 0)
+		(at 97 63 0)
 		(layer "F.SilkS")
 		(effects
@@
 	)
 	(segment
+		(start 93.5 60)
+		(end 104 70.5)
+		(width 0.2)
+		(layer "F.Cu")
+		(net "VIN-")
+	)
+	(segment
 		(start 132.325 84.85)
 		(end 131.5 85.675)
@@
 	)
 	(segment
-		(start 95.825 61.6)
-		(end 104.725 70.5)
-		(width 0.2)
-		(layer "F.Cu")
-		(net "VIN-")
-	)
-	(segment
 		(start 111.1 59.4)
 		(end 111.15 59.45)
@@
 	)
 	(segment
-		(start 95.825 59.325)
-		(end 95.825 61.6)
-		(width 0.2)
-		(layer "F.Cu")
-		(net "VIN-")
-	)
-	(segment
 		(start 111.25 74.6)
 		(end 110.525 75.325)
@@
 	)
 	(segment
+		(start 104 70.5)
+		(end 104.725 70.5)
+		(width 0.2)
+		(layer "F.Cu")
+		(net "VIN-")
+	)
+	(segment
 		(start 114.5 72)
 		(end 115 72)
@@
 	)
 	(segment
-		(start 99.425 59.325)
-		(end 99.425 60.925)
-		(width 0.2)
-		(layer "F.Cu")
-		(net "+3V3")
-	)
-	(segment
 		(start 139.715 90)
 		(end 141.5 90)
@@
 	)
 	(segment
-		(start 143.5 89.5)
-		(end 143.5 88)
-		(width 0.325)
+		(start 98.1 60)
+		(end 102.6 64.5)
+		(width 0.2)
 		(layer "F.Cu")
 		(net "+3V3")
 	)
 	(segment
-		(start 99.425 60.925)
-		(end 103 64.5)
-		(width 0.2)
+		(start 143.5 89.5)
+		(end 143.5 88)
+		(width 0.325)
 		(layer "F.Cu")
 		(net "+3V3")
@@
 	)
 	(segment
+		(start 102.6 64.5)
+		(end 103 64.5)
+		(width 0.2)
+		(layer "F.Cu")
+		(net "+3V3")
+	)
+	(segment
 		(start 134.5 71.5)
 		(end 131.5 71.5)
@@
 	)
 	(segment
-		(start 108.5 61.5)
-		(end 108.5 61.2)
-		(width 0.2)
-		(layer "F.Cu")
-		(net "IO2")
-	)
-	(segment
 		(start 109.2 62.65)
 		(end 109 62.85)
@@
 	(segment
 		(start 108.5 61.2)
-		(end 106.625 59.325)
+		(end 107.3 60)
+		(width 0.2)
+		(layer "F.Cu")
+		(net "IO2")
+	)
+	(segment
+		(start 108.5 61.5)
+		(end 108.5 61.2)
 		(width 0.2)
 		(layer "F.Cu")
@@
 	)
 	(segment
-		(start 107 61.5)
-		(end 104.825 59.325)
+		(start 104.2 61.5)
+		(end 102.7 60)
 		(width 0.2)
 		(layer "F.Cu")
@@
 	(segment
 		(start 107.5 61.5)
-		(end 107 61.5)
+		(end 104.2 61.5)
 		(width 0.2)
 		(layer "F.Cu")
@@
 		(width 0.2)
 		(layer "F.Cu")
-		(net "IO3")
-	)
-	(segment
-		(start 104.825 59.325)
-		(end 103.025 59.325)
-		(width 0.2)
-		(layer "F.Cu")

Commit message: Rah
Parts:
- R21: value 90K -> 91K
Changed lines of the file:
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@@
 			)
 		)
-		(property "Value" "90K"
+		(property "Value" "91K"
 			(at 0 1.43 0)
 			(layer "F.Fab")

Commit message: Change usb
Parts:
- removed J2, J5: USB_C_Receptacle_USB2.0_14P, Connector_USB:USB_C_Receptacle_XKB_U262-16XN-4BVC11
- added J6: USB_C_Receptacle_USB2.0_16P, Connector_USB:USB_C_Receptacle_GCT_USB4105-xx-A_16P_TopMnt_Horizontal, F.Cu at (94.5, 83.5)
- added J7: USB_C_Receptacle_USB2.0_16P, Connector_USB:USB_C_Receptacle_GCT_USB4105-xx-A_16P_TopMnt_Horizontal, F.Cu at (94.5, 94.5)
Routing:
- net VIN-: track 350.2 -> 374.0 mm, vias 12 -> 10
- net unconnected-(J5-SHIELD-PadSH): track 17.0 -> 0.00 mm
- net unconnected-(J2-SHIELD-PadSH): track 17.0 -> 0.00 mm
- net IO2: track 5.79 -> 7.92 mm
- net D-: track 66.3 -> 68.3 mm
- net Net-(D3-A): track 25.2 -> 26.2 mm
- net Net-(J7-CC2): track 18.6 -> 19.6 mm
- net Net-(J7-CC1): track 13.4 -> 14.4 mm
- net Net-(J6-CC2): track 9.70 -> 10.7 mm
- net Net-(J6-CC1): track 12.1 -> 13.1 mm
- net D+: track 69.5 -> 70.5 mm
- net Net-(D5-A): track 11.1 -> 12.0 mm
