File: ScholDigi.kicad_pcb (KiCad board)
At the start: 2 copper layers, 66 x 49 mm, 67 parts, among them J1 Conn_01x04, J3 Battery JST, J4 GPS Antenna coaxial, J6 USB_C_Receptacle_USB2.0_16P, J7 USB_C_Receptacle_USB2.0_16P, Q1 FS8205A, SW1 Boot Button, SW2 Reset Button, U1 ESP32-C6-MINI-1, U2 MAX-M10S, U3 TP4056-42-ESOP8, U4 DW01A, U5 TPS63060, U6 CP2102

Commit message: Inspirational quote
Other:
- board text added: "According to all laws of aerodynamics, the bumblebee cannot fly because its body weight is not the right proportion to its wingspan. But ignoring these laws the bee flies anyway."
