File: pcb/ScholDigi.kicad_pcb (KiCad board)
At the start: 2 copper layers, 66 x 49 mm, 67 parts, among them J1 Conn_01x04, J3 Battery JST, J4 GPS Antenna coaxial, J6 USB_C_Receptacle_USB2.0_16P, J7 USB_C_Receptacle_USB2.0_16P, Q1 FS8205A, SW1 Boot Button, SW2 Reset Button, U1 ESP32-C6-MINI-1, U2 MAX-M10S, U3 TP4056-42-ESOP8, U4 DW01A, U5 TPS63060, U6 CP2102

Commit message: Add pullups
Parts:
- added R23: 4.7K, Resistor_SMD:R_0603_1608Metric, F.Cu at (101.0, 65.0)
- added R24: 4.7K, Resistor_SMD:R_0603_1608Metric, F.Cu at (93.5, 57.0)
Routing:
- net IO3: track 10.0 -> 19.6 mm
- net +3V3: track 107.5 -> 116.7 mm
- net IO2: track 7.92 -> 16.0 mm, vias 2 -> 3

Commit message: more io
Parts:
- added J2: Conn_01x02, Connector_Wire:SolderWire-0.5sqmm_1x02_P4.6mm_D0.9mm_OD2.1mm, F.Cu at (93.1, 69.7)
Connections:
- U1 pad 28: unconnected-(U1-IO22-Pad28) -> Net-(J2-Pin_1)
- U1 pad 29: unconnected-(U1-IO23-Pad29) -> Net-(J2-Pin_2)
Routing:
- net Net-(J2-Pin_1): track 0.00 -> 44.6 mm, vias 0 -> 1
- net Net-(J2-Pin_2): track 0.00 -> 34.7 mm, vias 0 -> 1
Other:
- board text added: "IO22"
- board text added: "IO23"

Commit message: Clean up board
Routing:
- net Net-(J2-Pin_1): track 44.6 -> 43.5 mm
Changed lines of the file:
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@@
-	)
-	(segment
-		(start 93.105 68.605)
-		(end 93.105 69.675)
-		(width 0.2)
-		(layer "F.Cu")
-		(net "Net-(J2-Pin_1)")
 	)
 	(segment
@@
 	)
 	(segment
-		(start 120.375735 63.124265)
-		(end 120.375735 61.527206)
+		(start 97.75 58.25)
+		(end 91.6 64.4)
+		(width 0.2)
+		(layer "B.Cu")
+		(net "Net-(J2-Pin_1)")
+	)
+	(segment
+		(start 120.375735 61.527206)
+		(end 117.098529 58.25)
 		(width 0.2)
 		(layer "B.Cu")
@@
 	)
 	(segment
-		(start 93.105 68.605)
-		(end 93.105 69.675)
-		(width 0.2)
-		(layer "B.Cu")
-		(net "Net-(J2-Pin_1)")
-	)
-	(segment
-		(start 97.75 58.25)
-		(end 91.6 64.4)
+		(start 120.375735 63.124265)
+		(end 120.375735 61.527206)
 		(width 0.2)
 		(layer "B.Cu")
@@
 	(segment
 		(start 91.6 64.4)
-		(end 91.6 67.1)
+		(end 91.6 68.17)
 		(width 0.2)
 		(layer "B.Cu")
@@
 	)
 	(segment
-		(start 120.375735 61.527206)
-		(end 117.098529 58.25)
+		(start 91.6 68.17)
+		(end 93.105 69.675)
 		(width 0.2)
 		(layer "B.Cu")
-		(net "Net-(J2-Pin_1)")
-	)
-	(segment
-		(start 91.6 67.1)
-		(end 93.105 68.605)
-		(width 0.2)
-		(layer "B.Cu")
