File: pcb/ScholDigi.kicad_pcb (KiCad board)
At the start: 2 copper layers, 66 x 49 mm, 70 parts, among them J1 Conn_01x04, J2 Conn_01x02, J3 Battery JST, J4 GPS Antenna coaxial, J6 USB_C_Receptacle_USB2.0_16P, J7 USB_C_Receptacle_USB2.0_16P, Q1 FS8205A, SW1 Boot Button, SW2 Reset Button, U1 ESP32-C6-MINI-1, U2 MAX-M10S, U3 TP4056-42-ESOP8, U4 DW01A, U5 TPS63060, U6 CP2102

Commit message: Pullup boot button
Parts:
- added R25: 10K, Resistor_SMD:R_0603_1608Metric, F.Cu at (108.0, 77.7)
Routing:
- net +3V3: track 116.7 -> 122.7 mm, vias 6 -> 7
- net Net-(U1-IO9): track 19.8 -> 22.5 mm
Changed lines of the file:
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@@
 		)
 	)
+	(footprint "Resistor_SMD:R_0603_1608Metric"
+		(layer "F.Cu")
+		(at 107.995 77.745 180)
+		(descr "Resistor SMD 0603 (1608 Metric), square (rectangular) end terminal, IPC-7351 nominal, (Body size source: IPC-SM-782 page 72, https://www.pcb-3d.com/wordpress/wp-content/uploads/ipc-sm-782a_amendment_1_and_2.pdf)")
+		(tags "resistor")
+		(property "Reference" "R25"
+			(at 0 -1.43 0)
+			(layer "F.SilkS")
+			(effects
+				(font
+					(size 1 1)
+					(thickness 0.15)
+				)
+			)
+		)
+		(property "Value" "10K"
+			(at 0 1.43 0)
+			(layer "F.Fab")
+			(effects
+				(font
+					(size 1 1)
+					(thickness 0.15)
+				)
+			)
+		)
+		(property "Datasheet" ""
+			(at 0 0 0)
+			(layer "F.Fab")
+			(hide yes)
+			(effects
+				(font
+					(size 1.27 1.27)
+				)
+			)
+		)
+		(property "Description" "Resistor"
+			(at 0 0 0)
+			(layer "F.Fab")
+			(hide yes)
+			(effects
+				(font
+					(size 1.27 1.27)
+				)
+			)
+		)
+		(property "KiLib_Generator" "SMD_2terminal_chip_molded"
+			(at 0 0 0)
+			(layer "F.SilkS")
+			(hide yes)
+			(effects
+				(font
+					(size 1 1)
+					(thickness 0.15)
+				)
+			)
+		)
+		(property ki_fp_filters "R_*")
+		(sheetname "/")
+		(sheetfile "ScholDigi.kicad_sch")
+		(units
+			(unit
+				(name "A")
+				(pins "1" "2")
+			)
+		)
+		(attr smd)
+		(duplicate_pad_numbers_are_jumpers no)
+		(fp_line
+			(start -0.237258 0.5225)
+			(end 0.237258 0.5225)
+			(stroke
+				(width 0.12)
+				(type solid)
+			)
+			(layer "F.SilkS")
+		)
+		(fp_line
+			(start -0.237258 -0.5225)
+			(end 0.237258 -0.5225)
+			(stroke
+				(width 0.12)
+				(type solid)
+			)
+			(layer "F.SilkS")
+		)
+		(fp_rect
+			(start -1.48 -0.73)
+			(end 1.48 0.73)
+			(stroke
+				(width 0.05)
+				(type solid)
+			)
+			(fill no)
+			(layer "F.CrtYd")
+		)
+		(fp_rect
+			(start -0.8 -0.4125)
+			(end 0.8 0.4125)
+			(stroke
+				(width 0.1)
+				(type solid)
+			)
+			(fill no)
+			(layer "F.Fab")
+		)
+		(fp_text user "${REFERENCE}"
+			(at 0 0 0)
+			(layer "F.Fab")
+			(effects
+				(font
+					(size 0.4 0.4)
+					(thickness 0.06)
+				)
+			)
+		)
+		(pad "1" smd roundrect
+			(at -0.825 0 180)
+			(size 0.8 0.95)
+			(layers "F.Cu" "F.Mask" "F.Paste")
+			(roundrect_rratio 0.25)
+			(net "Net-(U1-IO9)")
+			(pintype "passive")
+		)
+		(pad "2" smd roundrect
+			(at 0.825 0 180)
+			(size 0.8 0.95)
+			(layers "F.Cu" "F.Mask" "F.Paste")
+			(roundrect_rratio 0.25)
+			(net "+3V3")
+			(pintype "passive")
+		)
+		(embedded_fonts no)
+		(model "${KICAD10_3DMODEL_DIR}/Resistor_SMD.3dshapes/R_0603_1608Metric.step"
+			(offset
+				(xyz 0 0 0)
+			)
+			(scale
+				(xyz 1 1 1)
+			)
+			(rotate
+				(xyz 0 0 0)
+			)
+		)
+	)
 	(footprint "Connector_Wire:SolderWire-0.5sqmm_1x02_P4.6mm_D0.9mm_OD2.1mm"
 		(layer "F.Cu")
@@
 	)
 	(segment
+		(start 107 76)
+		(end 107 77.575)
+		(width 0.2)
+		(layer "F.Cu")
+		(net "+3V3")
+	)
+	(segment
 		(start 140.5375 84.0375)
 		(end 140.5375 76.6125)
@@
 	)
 	(segment
+		(start 107 77.575)
+		(end 107.17 77.745)
+		(width 0.2)
+		(layer "F.Cu")
+		(net "+3V3")
+	)
+	(segment
 		(start 144 93)
 		(end 142.9 93)
@@
 	)
 	(via
+		(at 107 76)
+		(size 0.6)
+		(drill 0.3)
+		(layers "F.Cu" "B.Cu")
+		(net "+3V3")
+	)
+	(via
 		(at 144 95)
 		(size 0.6)
@@
 	)
 	(segment
+		(start 110.251471 73.6)
+		(end 110.075736 73.424264)
+		(width 0.2)
+		(layer "B.Cu")
+		(net "+3V3")
+	)
+	(segment
+		(start 110.075736 73.424264)
+		(end 107.5 76)
+		(width 0.2)
+		(layer "B.Cu")
+		(net "+3V3")
+	)
+	(segment
 		(start 117.048529 70.3)
 		(end 113.748529 73.6)
@@
 	)
 	(segment
-		(start 110.251471 73.6)
+		(start 110.075736 73.424264)
 		(end 103 66.348529)
 		(width 0.2)
@@
 	)
 	(segment
+		(start 107.5 76)
+		(end 107 76)
+		(width 0.2)
+		(layer "B.Cu")
+		(net "+3V3")
+	)
+	(segment
 		(start 143.5 94.5)
 		(end 144 95)
@@
 	)
 	(segment
+		(start 110.595 77.745)
+		(end 111.25 78.4)
+		(width 0.2)
+		(layer "F.Cu")
+		(net "Net-(U1-IO9)")
+	)
+	(segment
 		(start 118.15 79)
 		(end 119.5 79)
@@
 		(width 0.2)
 		(layer "F.Cu")
+		(net "Net-(U1-IO9)")
+	)
+	(segment
+		(start 108.82 77.745)
+		(end 110.595 77.745)
+		(width 0.2)
+		(layer "F.Cu")

Commit message: Fix pcb
Parts:
- added C16: 100uF, Capacitor_SMD:C_0603_1608Metric, F.Cu at (138.5, 76.5)
Connections:
- U2 pad 7: +3V3 -> Net-(U2-VCC)
- U2 pad 8: +3V3 -> Net-(U2-VCC)
Routing:
- net Net-(U2-VCC): track 0.00 -> 4.37 mm
- net +3V3: track 122.7 -> 124.0 mm

Commit message: Fix pcb
Parts:
- moved C16 1.80 mm to (139.5, 78.0), turned to 90 degrees
Routing:
- net +3V3: track 124.0 -> 122.6 mm
- net Net-(U2-VCC): track 4.37 -> 3.40 mm
Changed lines of the file:
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@@
 	(footprint "Capacitor_SMD:C_0603_1608Metric"
 		(layer "F.Cu")
-		(at 138.5 76.5 180)
+		(at 139.5 78 90)
 		(descr "Capacitor SMD 0603 (1608 Metric), square (rectangular) end terminal, IPC-7351 nominal, (Body size source: IPC-SM-782 page 76, https://www.pcb-3d.com/wordpress/wp-content/uploads/ipc-sm-782a_amendment_1_and_2.pdf)")
 		(tags "capacitor")
 		(property "Reference" "C16"
-			(at 0 -1.43 0)
+			(at 1.5 -2.5 0)
 			(layer "F.SilkS")
 			(effects
@@
 		)
 		(property "Value" "100uF"
-			(at 0 1.43 0)
+			(at -1.5 -1.5 90)
 			(layer "F.Fab")
 			(effects
@@
 		)
 		(property "Datasheet" ""
-			(at 0 0 0)
+			(at 0 0 90)
 			(layer "F.Fab")
 			(hide yes)
@@
 		)
 		(property "Description" "Unpolarized capacitor"
-			(at 0 0 0)
+			(at 0 0 90)
 			(layer "F.Fab")
 			(hide yes)
@@
 		)
 		(property "KiLib_Generator" "SMD_2terminal_chip_molded"
-			(at 0 0 0)
+			(at 0 0 90)
 			(layer "F.SilkS")
 			(hide yes)
@@
 		(duplicate_pad_numbers_are_jumpers no)
 		(fp_line
-			(start -0.14058 0.51)
-			(end 0.14058 0.51)
+			(start -0.14058 -0.51)
+			(end 0.14058 -0.51)
 			(stroke
 				(width 0.12)
@@
 		)
 		(fp_line
-			(start -0.14058 -0.51)
-			(end 0.14058 -0.51)
+			(start -0.14058 0.51)
+			(end 0.14058 0.51)
 			(stroke
 				(width 0.12)
@@
 		)
 		(fp_text user "${REFERENCE}"
-			(at 0 0 0)
+			(at 0 0 90)
 			(layer "F.Fab")
 			(effects
@@
 		)
 		(pad "1" smd roundrect
-			(at -0.775 0 180)
+			(at -0.775 0 90)
 			(size 0.9 0.95)
 			(layers "F.Cu" "F.Mask" "F.Paste")
@@
 		)
 		(pad "2" smd roundrect
-			(at 0.775 0 180)
+			(at 0.775 0 90)
 			(size 0.9 0.95)
 			(layers "F.Cu" "F.Mask" "F.Paste")
@@
 	)
 	(segment
-		(start 140.5375 84.0375)
-		(end 140.5375 76.6125)
-		(width 0.325)
-		(layer "F.Cu")
-		(net "+3V3")
-	)
-	(segment
 		(start 93.075 57)
 		(end 96.075 60)
@@
 	)
 	(segment
-		(start 140.425 76.5)
-		(end 140.5375 76.6125)
+		(start 143.5 88)
+		(end 144 87.5)
 		(width 0.325)
 		(layer "F.Cu")
@@
 	)
 	(segment
-		(start 143.5 88)
-		(end 144 87.5)
-		(width 0.325)
+		(start 138.5 76)
+		(end 138.15 75.65)
+		(width 0.2)
 		(layer "F.Cu")
 		(net "+3V3")
@@
 	)
 	(segment
+		(start 140.5375 79.8125)
+		(end 140.5375 84.0375)
+		(width 0.2)
+		(layer "F.Cu")
+		(net "+3V3")
+	)
+	(segment
 		(start 144 95)
 		(end 145.675 95)
@@
 	)
 	(segment
-		(start 140.5375 76.6125)
-		(end 140.9 76.25)
-		(width 0.325)
-		(layer "F.Cu")
-		(net "+3V3")
-	)
-	(segment
 		(start 141.8 75.15)
 		(end 138.15 75.15)
@@
 	)
 	(segment
-		(start 141.8 75.15)
-		(end 141.8 76.25)
-		(width 0.2)
-		(layer "F.Cu")
-		(net "+3V3")
-	)
-	(segment
 		(start 101.675 65.825)
 		(end 103 64.5)
@@
 	)
 	(segment
+		(start 138.5 77.775)
+		(end 138.5 76)
+		(width 0.2)
+		(layer "F.Cu")
+		(net "+3V3")
+	)
+	(segment
 		(start 96.075 60)
 		(end 98.1 60)
@@
 	)
 	(segment
+		(start 138.15 75.65)
+		(end 138.15 75.15)
+		(width 0.2)
+		(layer "F.Cu")
+		(net "+3V3")
+	)
+	(segment
 		(start 145.675 93)
 		(end 144 93)
@@
 	)
 	(segment
-		(start 139.275 76.5)
-		(end 140.425 76.5)
-		(width 0.325)
-		(layer "F.Cu")
-		(net "+3V3")
-	)
-	(segment
 		(start 101 65.825)
 		(end 101.675 65.825)
@@
 	)
 	(segment
-		(start 140.9 76.25)
-		(end 141.8 76.25)
-		(width 0.325)
+		(start 139.5 78.775)
+		(end 138.5 77.775)
+		(width 0.2)
 		(layer "F.Cu")
 		(net "+3V3")
@@
 		(net "+3V3")
 	)
+	(segment
+		(start 139.5 78.775)
+		(end 140.5375 79.8125)
+		(width 0.2)
+		(layer "F.Cu")
+		(net "+3V3")
+	)
 	(via
 		(at 103 64.5)
@@
 	)
 	(segment
-		(start 138.1375 75.6125)
-		(end 141.3375 75.6125)
-		(width 0.325)
-		(layer "F.Cu")
-		(net "Net-(U2-VCC)")
-	)
-	(segment
-		(start 141.3375 75.6125)
-		(end 141.3375 75.725)
-		(width 0.325)
+		(start 141.8 76.25)
+		(end 141.8 75.55)
+		(width 0.2)
 		(layer "F.Cu")
 		(net "Net-(U2-VCC)")
 	)
 	(segment
-		(start 137.725 76.025)
-		(end 138.1375 75.6125)
-		(width 0.325)
+		(start 140.475 76.25)
+		(end 141.8 76.25)
+		(width 0.2)
 		(layer "F.Cu")
 		(net "Net-(U2-VCC)")
 	)
 	(segment
-		(start 137.725 76.5)
-		(end 137.725 76.025)
-		(width 0.325)
+		(start 139.5 77.225)
+		(end 140.475 76.25)
+		(width 0.2)
 		(layer "F.Cu")
 		(net "Net-(U2-VCC)")

Commit message: Fix GPS
Parts:
- moved C16 1.80 mm to (138.5, 76.5), turned to 180 degrees
Connections:
- C16 pad 2: Net-(U2-VCC) -> VIN-
- U2 pad 7: Net-(U2-VCC) -> +3V3
- U2 pad 8: Net-(U2-VCC) -> +3V3
Routing:
- net VIN-: track 374.0 -> 385.4 mm, vias 10 -> 12
- net Net-(U2-VCC): track 3.40 -> 0.00 mm
- net +3V3: track 122.6 -> 124.1 mm

Commit message: Rah
Parts:
- C16: value 100uF -> 100nF
Changed lines of the file:
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@@
 			)
 		)
-		(property "Value" "100uF"
-			(at 0 1.43 0)
+		(property "Value" "100nF"
+			(at 3.5 0.5 0)
 			(layer "F.Fab")
 			(effects

Commit message: BOM
Parts:
- moved C16 1.12 mm to (139.0, 75.5), turned to 90 degrees
Routing:
- net VIN-: track 385.4 -> 382.5 mm
- net +3V3: track 124.1 -> 123.0 mm
Changed lines of the file:
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@@
 		(tags "resistor")
 		(property "Reference" "R6"
-			(at -2.55 0.05 0)
+			(at -1 -1.5 0)
 			(layer "F.SilkS")
 			(effects
@@
 		(tags "resistor")
 		(property "Reference" "R4"
-			(at 1 1.5 180)
+			(at 2 0 180)
 			(layer "F.SilkS")
 			(effects
@@
 	(footprint "Capacitor_SMD:C_0603_1608Metric"
 		(layer "F.Cu")
-		(at 138.5 76.5 180)
+		(at 139 75.5 90)
 		(descr "Capacitor SMD 0603 (1608 Metric), square (rectangular) end terminal, IPC-7351 nominal, (Body size source: IPC-SM-782 page 76, https://www.pcb-3d.com/wordpress/wp-content/uploads/ipc-sm-782a_amendment_1_and_2.pdf)")
 		(tags "capacitor")
 		(property "Reference" "C16"
-			(at 0 -1.43 0)
+			(at 0 -1.43 90)
 			(layer "F.SilkS")
 			(effects
@@
 		)
 		(property "Value" "100nF"
-			(at 3.5 0.5 0)
+			(at 3.5 0.5 90)
 			(layer "F.Fab")
 			(effects
@@
 		)
 		(property "Datasheet" ""
-			(at 0 0 0)
+			(at 0 0 90)
 			(layer "F.Fab")
 			(hide yes)
@@
 		)
 		(property "Description" "Unpolarized capacitor"
-			(at 0 0 0)
+			(at 0 0 90)
 			(layer "F.Fab")
 			(hide yes)
@@
 		)
 		(property "KiLib_Generator" "SMD_2terminal_chip_molded"
-			(at 0 0 0)
+			(at 0 0 90)
 			(layer "F.SilkS")
 			(hide yes)
@@
 		(duplicate_pad_numbers_are_jumpers no)
 		(fp_line
-			(start -0.14058 0.51)
-			(end 0.14058 0.51)
+			(start -0.14058 -0.51)
+			(end 0.14058 -0.51)
 			(stroke
 				(width 0.12)
@@
 		)
 		(fp_line
-			(start -0.14058 -0.51)
-			(end 0.14058 -0.51)
+			(start -0.14058 0.51)
+			(end 0.14058 0.51)
 			(stroke
 				(width 0.12)
@@
 		)
 		(fp_text user "${REFERENCE}"
-			(at 0 0 0)
+			(at 0 0 90)
 			(layer "F.Fab")
 			(effects
@@
 		)
 		(pad "1" smd roundrect
-			(at -0.775 0 180)
+			(at -0.775 0 90)
 			(size 0.9 0.95)
 			(layers "F.Cu" "F.Mask" "F.Paste")
@@
 		)
 		(pad "2" smd roundrect
-			(at 0.775 0 180)
+			(at 0.775 0 90)
 			(size 0.9 0.95)
 			(layers "F.Cu" "F.Mask" "F.Paste")
@@
 		)
 		(property "Value" "4.7K"
-			(at 0 1.43 0)
+			(at 0 3 0)
 			(layer "F.Fab")
 			(effects
@@
 	)
 	(segment
-		(start 137.725 75.725)
-		(end 137 75)
-		(width 0.2)
-		(layer "F.Cu")
-		(net "VIN-")
-	)
-	(segment
 		(start 117.55 73.55)
 		(end 115.5 71.5)
@@
 	)
 	(segment
-		(start 137.725 76.5)
-		(end 137.725 75.725)
-		(width 0.2)
-		(layer "F.Cu")
-		(net "VIN-")
-	)
-	(segment
 		(start 133.275 73.45)
 		(end 131.7 73.45)
@@
 	)
 	(segment
+		(start 139 74)
+		(end 140 73)
+		(width 0.2)
+		(layer "F.Cu")
+		(net "VIN-")
+	)
+	(segment
 		(start 111.25 74.6)
 		(end 110.525 75.325)
@@
 	)
 	(segment
+		(start 139 74.725)
+		(end 139 74)
+		(width 0.2)
+		(layer "F.Cu")
+		(net "VIN-")
+	)
+	(segment
 		(start 114.5 72)
 		(end 115 72)
@@
 	)
 	(via
-		(at 137 75)
+		(at 114.5 72)
 		(size 0.6)
 		(drill 0.3)
@@
 	)
 	(via
-		(at 114.5 72)
+		(at 110 97.5)
 		(size 0.6)
 		(drill 0.3)
@@
 	)
 	(via
-		(at 110 97.5)
+		(at 140 68.5)
 		(size 0.6)
 		(drill 0.3)
@@
 	)
 	(via
-		(at 140 68.5)
+		(at 140 73)
 		(size 0.6)
 		(drill 0.3)
@@
 	)
 	(segment
-		(start 137 75)
-		(end 140 72)
+		(start 140 73)
+		(end 140 68.5)
 		(width 0.2)
 		(layer "B.Cu")
@@
 	)
 	(segment
-		(start 140 72)
-		(end 140 68.5)
-		(width 0.2)
-		(layer "B.Cu")
-		(net "VIN-")
-	)
-	(segment
 		(start 135 84.5)
 		(end 138 87.5)
@@
 	)
 	(segment
-		(start 140.5375 84.0375)
-		(end 140.5375 77.7625)
-		(width 0.325)
-		(layer "F.Cu")
-		(net "+3V3")
-	)
-	(segment
 		(start 107 76)
 		(end 107 77.575)
@@
 	)
 	(segment
-		(start 144 87.5)
-		(end 140.5375 84.0375)
-		(width 0.325)
+		(start 98.1 60)
+		(end 102.6 64.5)
+		(width 0.2)
 		(layer "F.Cu")
 		(net "+3V3")
 	)
 	(segment
-		(start 98.1 60)
-		(end 102.6 64.5)
+		(start 134.75 71.5)
+		(end 131.5 71.5)
 		(width 0.2)
 		(layer "F.Cu")
@@
 	)
 	(segment
-		(start 141.8 75.15)
-		(end 138.15 75.15)
+		(start 102.6 64.5)
+		(end 103 64.5)
 		(width 0.2)
 		(layer "F.Cu")
@@
 	)
 	(segment
-		(start 102.6 64.5)
-		(end 103 64.5)
+		(start 134.75 72.025)
+		(end 134.75 71.5)
 		(width 0.2)
 		(layer "F.Cu")
@@
 	)
 	(segment
-		(start 134.5 71.5)
-		(end 131.5 71.5)
+		(start 139 76.275)
+		(end 134.75 72.025)
 		(width 0.2)
 		(layer "F.Cu")
@@
 	)
 	(segment
-		(start 138.15 75.15)
-		(end 134.5 71.5)
+		(start 107 77.575)
+		(end 107.17 77.745)
 		(width 0.2)
 		(layer "F.Cu")
@@
 	)
 	(segment
-		(start 107 77.575)
-		(end 107.17 77.745)
+		(start 141.8 76.25)
+		(end 139.025 76.25)
 		(width 0.2)
 		(layer "F.Cu")
@@
 	)
 	(segment
+		(start 139.025 76.25)
+		(end 139 76.275)
+		(width 0.2)
+		(layer "F.Cu")
+		(net "+3V3")
+	)
+	(segment
 		(start 96.075 60)
 		(end 98.1 60)
@@
 	)
 	(segment
+		(start 139 76.275)
+		(end 139 80.898962)
+		(width 0.2)
+		(layer "F.Cu")
+		(net "+3V3")
+	)
+	(segment
+		(start 144 85.898962)
+		(end 139.275 81.173962)
+		(width 0.325)
+		(layer "F.Cu")
+		(net "+3V3")
+	)
+	(segment
 		(start 145.675 93)
 		(end 144 93)
@@
 	)
 	(segment
-		(start 140.5375 77.7625)
-		(end 139.275 76.5)
-		(width 0.325)
+		(start 139 80.898962)
+		(end 139.275 81.173962)
+		(width 0.2)
 		(layer "F.Cu")
 		(net "+3V3")
@@
 	)
 	(segment
-		(start 144 93)
-		(end 143.5 93)
+		(start 144 87.5)
+		(end 144 85.898962)
 		(width 0.325)
 		(layer "F.Cu")
@@
 	)
 	(segment
-		(start 142.9 93)
-		(end 142.5 92.6)
+		(start 144 93)
+		(end 143.5 93)
 		(width 0.325)
 		(layer "F.Cu")
@@
 	)
 	(segment
-		(start 139.275 76.5)
-		(end 141.55 76.5)
-		(width 0.2)
+		(start 142.9 93)
+		(end 142.5 92.6)
+		(width 0.325)
 		(layer "F.Cu")
 		(net "+3V3")
